File: c64-eeprom.kicad_pcb (KiCad board)
At the start: 2 copper layers, 21.6 x 36.1 mm, 8 parts, among them J1 Conn_01x12_Pin, J2 Conn_01x12_Pin

Commit message: Added silkscreen to top to indicate compatible eeproms.
Other:
- board text added: "AT28C64 AT28C256"
- board text added: "C64"
Changed lines of the file:
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@@
       (plot_on_all_layers_selection 0x0000000_00000000)
       (disableapertmacros false)
-      (usegerberextensions false)
-      (usegerberattributes true)
-      (usegerberadvancedattributes true)
-      (creategerberjobfile true)
+      (usegerberextensions true)
+      (usegerberattributes false)
+      (usegerberadvancedattributes false)
+      (creategerberjobfile false)
       (dashed_line_dash_ratio 12.000000)
       (dashed_line_gap_ratio 3.000000)
@@
       (psa4output false)
       (plotreference true)
-      (plotvalue true)
+      (plotvalue false)
       (plotinvisibletext false)
       (sketchpadsonfab false)
-      (subtractmaskfromsilk false)
+      (subtractmaskfromsilk true)
       (outputformat 1)
       (mirror false)
-      (drillshape 1)
+      (drillshape 0)
       (scaleselection 1)
-      (outputdirectory "")
+      (outputdirectory "plots/")
     )
   )
@@
     (pad "28" smd rect (at 8.255 -16.51) (size 3.1 1.6) (layers "F.Cu" "F.Paste" "F.Mask")
       (net 24 "VCC") (pinfunction "VCC") (pintype "power_in"))
-    (model "${KICAD6_3DMODEL_DIR}/Package_DIP.3dshapes/DIP-28_W16.51mm_SMDSocket.wrl"
+    (model "${KICAD6_3DMODEL_DIR}/Package_DIP.3dshapes/DIP-28_W16.51mm_SMDSocket.wrl" hide
       (offset (xyz 0 0 0))
       (scale (xyz 1 1 1))
@@
     (effects (font (size 1 1) (thickness 0.2) bold) (justify right mirror))
   )
+  (gr_text "AT28C64\nAT28C256" (at 140.208 74.803 90) (layer "F.SilkS")
+    (effects (font (size 2 2) (thickness 0.4) bold))
+  )
+  (gr_text "C64" (at 140.208 90.17) (layer "F.SilkS")
+    (effects (font (size 2 2) (thickness 0.4) bold))
+  )
   (segment (start 132.08 63.5) (end 136.652 63.5) (width 0.5) (layer "F.Cu") (net 1))

Commit message: Fix disconnected jumper pad, A12.
Connections:
- JP3 pad 2: unconnected-(JP3-B-Pad2) -> GND
Changed lines of the file:
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@@
   (net 26 "Net-(JP2-C)")
   (net 27 "Net-(JP3-A)")
-  (net 28 "unconnected-(JP3-B-Pad2)")
-  (net 29 "Net-(JP4-B)")
+  (net 28 "Net-(JP4-B)")
   (footprint "Package_DIP:DIP-28_W16.51mm_SMDSocket_LongPads" (layer "F.Cu")
     (at 140.335 74.93)
@@
       (net 19 "Net-(J2-Pin_7)") (pinfunction "A10") (pintype "input"))
     (pad "22" smd rect (at 8.255 -1.27) (size 3.1 1.6) (layers "F.Cu" "F.Paste" "F.Mask")
-      (net 29 "Net-(JP4-B)") (pinfunction "OE") (pintype "input"))
+      (net 28 "Net-(JP4-B)") (pinfunction "OE") (pintype "input"))
     (pad "23" smd rect (at 8.255 -3.81) (size 3.1 1.6) (layers "F.Cu" "F.Paste" "F.Mask")
       (net 18 "Net-(J2-Pin_6)") (pinfunction "A11") (pintype "input"))
@@
       ))
     (pad "2" smd custom (at 0.65 0 180) (size 1 0.5) (layers "B.Cu" "B.Mask")
-      (net 28 "unconnected-(JP3-B-Pad2)") (pinfunction "B") (pintype "passive") (zone_connect 2)
+      (net 12 "GND") (pinfunction "B") (pintype "passive") (zone_connect 2)
       (options (clearance outline) (anchor rect))
       (primitives
@@
       (stroke (width 0.05) (type solid)) (layer "B.CrtYd"))
     (pad "1" smd custom (at -0.65 0 180) (size 1 0.5) (layers "B.Cu" "B.Mask")
-      (net 29 "Net-(JP4-B)") (pinfunction "A") (pintype "passive") (zone_connect 2)
+      (net 28 "Net-(JP4-B)") (pinfunction "A") (pintype "passive") (zone_connect 2)
       (options (clearance outline) (anchor rect))
       (primitives
@@
       (net 21 "Net-(J2-Pin_9)") (pinfunction "C") (pintype "passive"))
     (pad "3" smd custom (at 1.3 0 270) (size 1 0.5) (layers "B.Cu" "B.Mask")
-      (net 29 "Net-(JP4-B)") (pinfunction "B") (pintype "passive") (zone_connect 2)
+      (net 28 "Net-(JP4-B)") (pinfunction "B") (pintype "passive") (zone_connect 2)
       (options (clearance outline) (anchor rect))
       (primitives
@@
   (segment (start 138.938 64.008) (end 138.938 68.453) (width 0.5) (layer "B.Cu") (net 27))
   (segment (start 139.573 64.008) (end 140.335 64.77) (width 0.5) (layer "B.Cu") (net 27))
-  (segment (start 146.304 73.66) (end 148.59 73.66) (width 0.5) (layer "F.Cu") (net 29))
-  (segment (start 144.78 72.136) (end 146.304 73.66) (width 0.5) (layer "F.Cu") (net 29))
-  (segment (start 141.732 72.136) (end 144.78 72.136) (width 0.5) (layer "F.Cu") (net 29))
-  (via (at 141.732 72.136) (size 0.8) (drill 0.4) (layers "F.Cu" "B.Cu") (net 29))
-  (segment (start 140.462 73.406) (end 140.208 73.406) (width 0.5) (layer "B.Cu") (net 29))
-  (segment (start 141.732 72.136) (end 140.462 73.406) (width 0.5) (layer "B.Cu") (net 29))
-  (segment (start 141.732 72.136) (end 141.732 68.767) (width 0.5) (layer "B.Cu") (net 29))
-  (segment (start 141.732 68.767) (end 140.335 67.37) (width 0.5) (layer "B.Cu") (net 29))
+  (segment (start 146.304 73.66) (end 148.59 73.66) (width 0.5) (layer "F.Cu") (net 28))
+  (segment (start 144.78 72.136) (end 146.304 73.66) (width 0.5) (layer "F.Cu") (net 28))
+  (segment (start 141.732 72.136) (end 144.78 72.136) (width 0.5) (layer "F.Cu") (net 28))
+  (via (at 141.732 72.136) (size 0.8) (drill 0.4) (layers "F.Cu" "B.Cu") (net 28))
+  (segment (start 140.462 73.406) (end 140.208 73.406) (width 0.5) (layer "B.Cu") (net 28))
+  (segment (start 141.732 72.136) (end 140.462 73.406) (width 0.5) (layer "B.Cu") (net 28))
+  (segment (start 141.732 72.136) (end 141.732 68.767) (width 0.5) (layer "B.Cu") (net 28))
+  (segment (start 141.732 68.767) (end 140.335 67.37) (width 0.5) (layer "B.Cu") (net 28))
   (zone (net 12) (net_name "GND") (layers "F&B.Cu") (hatch edge 0.5)
     (connect_pads (clearance 0.5))
