File: c64-eeprom.kicad_sch (KiCad schematic)
At the start: 9 parts, among them J1 Conn_01x12_Pin, J2 Conn_01x12_Pin

Commit message: Fix disconnected jumper pad, A12.
Connections:
- net GND: now also JP3.2 (B)
Changed lines of the file:
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@@
+    (stroke (width 0) (type default))
+  )
+  (wire (pts (xy 184.15 128.27) (xy 184.15 130.81))
     (stroke (width 0) (type default))
   )
